File: UpperArmBoard/upperArm.brd (EAGLE design)
At the start: 100 x 80 mm, 2 parts

Commit message: nearly done!
Parts:
- added 3V, 5V, 5VG, BQ_USB_VBUS, HYD_COM1, HYD_COM2, HYD_RX_AMP, HYD_TX_SIG, SCLG, SCL_3V, SCL_5V, SDAG, SDA_3V, SDA_5V, TPA_L+, TPA_L-, TPA_R+, TPA_R-, TP_TXRX, VBAT, VBAT1: TPB1,27, testpad:B1,27
- added C1, C4, C6: 1uF, rcl:C0805
- added C10: 10uF, microbuilder:0805
- added C16, C17: 9pF, rcl:C0805
- added C2, C3: 10uF, rcl:C0805
- added C21, C5: 0.1uF, rcl:C0805
- added C7: 0.1µF, microbuilder:0805
- added C8: 0.01uF, microbuilder:0805
- added C9: 100pF, microbuilder:0805
- added D1, D10, D11, D13, D2, D3, D4, D5, D6, D7, D8, D9: WS2812_5050, SparkFun-LED:WS2812-5X5-4PIN
- added D12: SK34AQ-LTP, SamacSys_Parts:DIOM5226X244N
- added FB2, FB3: BLM18PG471SN1D, SamacSys_Parts:BLM18SP221SN1B
- added IC1: LTC4311CSC6#TRPBF, SamacSys_Parts:SOT65P210X100-6N
- added IC2: MAX17048G+T10, SamacSys_Parts:SON50P200X200X80-9N
- added IC3: PAM8904EGPR, SamacSys_Parts:QFN40P200X200X80-13N
- added IC4: DS04-254-2-02BK-SMT, SamacSys_Parts:DS04254202BKSMT
- added J2, J3, J4: 1727052, SamacSys_Parts:1727052
- added JP11, JP12, JP13, JP7: (no value), pinhead:1X01
- added JP14, JP2, JP3, JP8: JUMPER-SMT_3_1-NC_TRACE_NO-SILK, SparkFun-Jumpers:SMT-JUMPER_3_1-NC_TRACE_NO-SILK
- added JP4: (no value), pinhead:1X06
- added JP5, JP6, JP9: JUMPER-SMT_2_NC_TRACE_NO-SILK, SparkFun-Jumpers:SMT-JUMPER_2_NC_TRACE_NO-SILK
- added K1, K2: G6K-2P-Y-DC5, SamacSys_Parts:G6K2PYDC12
- added LED2: RED, led:CHIP-LED0805
- added Q1, Q2: CSD17575Q3, SamacSys_Parts:CSD16327
- added Q3, Q4: BSS138, microbuilder:SOT23-WIDE
- added R1, R17, R18, R2, R3, R32, R4, R5: 10k, rcl:R0805
- added R10, R9: 1M, microbuilder:0805
- added R11: 22K, microbuilder:0805
- added R12: 3386P-1-104LF, 3386P-1-104LF:POT_3386P
- added R13: 100, rcl:R0603
- added R14, R23: 220, rcl:R0805
- added R27: 100k, rcl:R0805
- added R29: 100, rcl:R0805
- added R6, R7, R8: 1K, microbuilder:0805
- added S1: GPTS203211B, SamacSys_Parts:GPTS203211B
- added U$11, U$14, U$15, U$16, U$17, U$18, U$19: MOUNTINGHOLE2.5, microbuilder:MOUNTINGHOLE_2.5_PLATED
- added U$7: (no value), pinhead:1X10
- added U1: MAX4466EXK+T, microbuilder:SC70-5
- added U8: BNO055, BNO055:LGA28R50P4X10_380X520X100
- added VR2: PT01-D115D-B103, SamacSys_Parts:PT01D115DB103
- added Y1: NDK_NX3215SA-32.768K-STD-MUA-9, NDK - NX3215SA-32.768K-STD-MUA-8:NDK_NX3215SA-32.768K-STD-MUA-8_0
- moved JP1 82.1 mm to (66.0, 60.7), turned to 270 degrees
- moved U$1 8.36 mm to (18.6, 60.7)
Connections:
- removed net BQ_LIPO_IN: JP1.10
- new net 3.3V: 3V.TP, C5.1, J2.2, JP14.3, JP8.1, Q3.1, Q4.1, R2.2, R3.2, R32.2, U$1.3V, U$7.10, U8.28, U8.3, VR2.1
- new net 5V: 5V.TP, C3.1, D1.VCC, D10.VCC, D11.VCC, D13.VCC, D2.VCC, D3.VCC, D4.VCC, D5.VCC, D6.VCC, D7.VCC, D8.VCC, D9.VCC, IC1.1, IC3.12, IC4.3, IC4.4, J3.2, JP14.1, JP4.1, K1.1, K2.1, R1.2, R17.2, R18.2, U$1.5V, U$7.1
- new net AGND: C10.2, C7.2, FB2.1, R9.1, U1.2
- new net AVCC: FB3.1, R10.2, R7.2, U1.5
- new net BONECOND_+: J2.5, JP7.1, TPA_L+.TP
- new net BONECOND_-: J2.6, JP11.1, TPA_L-.TP
- new net HYD_COM1: HYD_COM1.TP, J2.3, K1.3
- new net HYD_COM2: HYD_COM2.TP, J2.4, K2.3
- new net HYD_RX_IN1: C8.1, K1.2, R6.1
- new net HYD_RX_IN2: K2.2
- new net HYD_RX_INPUT: C9.1, HYD_RX_AMP.TP, R12.1, R12.2, U$1.MIC, U1.4
- new net HYD_TX_OUT1: IC3.6, K1.4
- new net HYD_TX_OUT2: IC3.7, K2.4
- new net HYD_TX_SIG: HYD_TX_SIG.TP, IC3.3, U$1.3
- new net IMU_CLK1: C16.2, U8.27, Y1.1
- new net IMU_CLK2: C17.2, U8.26, Y1.2
- new net LED_BRIDGE: D6.DI, D8.DO
- new net LED_DIN: R13.1, U$1.2
- new net LED_DOUT: D11.DO, J3.5
- new net N$1: IC1.3, R1.1
- new net N$11: IC3.13, JP9.2
- new net N$12: IC3.1, IC4.2, R4.2
- new net N$13: IC3.2, IC4.1, R5.1
- new net N$15: FB3.2, JP14.2
- new net N$16: C7.1, R6.2, R7.1
- new net N$17: C8.2, R10.1, R9.2, U1.1
- new net N$18: D1.DI, D13.DO
- new net N$19: C9.2, R11.1, R8.2, U1.3
- new net N$20: C10.1, R8.1
- new net N$21: R11.2, R12.3
- new net N$24: D12.2, J4.3
- new net N$25: D2.DO, D3.DI
- new net N$26: D3.DO, D4.DI
- new net N$27: D4.DO, D5.DI
- new net N$28: D5.DO, D8.DI
- new net N$29: D7.DO, D9.DI
- new net N$30: D10.DI, D9.DO
- new net N$31: D10.DO, D11.DI
- new net N$32: JP6.2, U$7.7
- new net N$37: C21.2, U8.9
- new net N$4: D6.DO, D7.DI
- new net N$40: R32.1, U8.4
- new net N$5: IC2.2, JP8.2
- new net N$6: Q2.4, R14.2
- new net N$7: C2.1, IC3.10
- new net N$81: Q1.4, R23.2
- new net N$82: LED2.A, R29.1
- new net NC_BCLK: U$1.21
- new net NC_DIN: U$1.7
- new net NC_DOUT: U$1.8
- new net NC_LRCLK: U$1.20
- new net NC_MCLK: U$1.23
- new net NC_MEMCS: U$1.6
- new net NC_MISO: U$1.12
- new net NC_MOSI: U$1.11
- new net NC_SCK: U$1.13
- new net NC_SDCS: U$1.10
- new net NC_VOL: U$1.15
- new net PAM_CN1: C4.2, IC3.4
- new net PAM_CN2: C6.2, IC3.8
- new net PAM_CP1: C4.1, IC3.9
- new net PAM_CP2: C6.1, IC3.11
- new net PB1K_EN: J4.5, JP4.4, S1.2
- new net PB1K_LB: JP4.3
- new net SCL_3V: IC2.7, JP3.2, Q4.2, R3.1, SCL_3V.TP, U$7.8, U8.19
- new net SCL_5V: IC1.6, J3.4, Q4.3, R18.1, SCL_5V.TP
- new net SDA_3V: IC2.8, JP2.2, Q3.2, R2.1, SDA_3V.TP, U$7.9, U8.20
- new net SDA_5V: IC1.4, J3.3, Q3.3, R17.1, SDA_5V.TP
- new net TPA_L+: U$1.OUTL, U$7.6
- new net TPA_R+: U$1.OUTR, U$7.5
- new net TPA_SHDN: U$7.3
- new net TXRX_OUT1: K1.8, Q1.5, Q1.6, Q1.7, Q1.8
- new net TXRX_OUT2: K2.8, Q2.5, Q2.6, Q2.7, Q2.8
- new net TXRX_RELAY: R14.1, R23.1, R27.1, R29.2, TP_TXRX.TP
- new net VBAT: C1.1, IC2.3, J4.1, JP1.10, JP8.3, VBAT.TP
- new net VOL_POT_SIG: J2.1, U$1.14, VR2.2
- net 3.3VI2C_SCL0: now also JP3.3
- net 3.3VI2C_SCL1: now also JP3.1
- net 3.3VI2C_SDA0: now also JP2.3
- net 3.3VI2C_SDA1: now also JP2.1
- net BQ_LOAD_OUT: now also JP4.6
- net BQ_USB_VBUS: now also BQ_USB_VBUS.TP, D12.1
- net GND: now also 5VG.TP, C1.2, C16.1, C17.1, C2.2, C21.1, C3.2, C5.2, D1.GND, D10.GND, D11.GND, D13.GND, D2.GND, D3.GND, D4.GND, D5.GND, D6.GND, D7.GND, D8.GND, D9.GND, FB2.2, IC1.2, IC1.5, IC2.1, IC2.4, IC2.6, IC2.9, IC3.5, J3.1, J3.6, J4.2, J4.4, J4.6, JP4.2, JP4.5, JP5.1, JP6.1, JP9.1, LED2.C, Q1.1, Q1.2, Q1.3, Q2.1, Q2.2, Q2.3, R27.2, R4.1, R5.2, S1.1, SCLG.TP, SDAG.TP, U$1.G, U$1.GND_MIC, U$1.INGND1, U$1.INGND2, U$1.OUTGND, U$7.2, U8.10, U8.15, U8.16, U8.17, U8.18, U8.2, U8.25, U8.5, U8.6, VBAT1.TP, VR2.3
- net N$10: now also D1.DO, D2.DI; no longer U$1.VOL_3.3V
- net N$2: now also JP12.1, TPA_R+.TP; no longer U$1.5V
- net N$3: now also JP13.1, TPA_R-.TP; no longer U$1.G
- net N$8: now also D13.DI, R13.2; no longer U$1.VOL_GND
- net N$9: now also JP5.2, U$7.4; no longer U$1.VOL
Routing:
- net GND: track 0.00 -> 173.4 mm
- net 5V: track 0.00 -> 138.4 mm
- net N$24: track 0.00 -> 57.6 mm, vias 0 -> 4
- net HYD_RX_INPUT: track 0.00 -> 48.1 mm
- net VBAT: track 0.00 -> 33.4 mm
- net SDA_5V: track 0.00 -> 27.8 mm
- net 3.3V: track 0.00 -> 25.3 mm
- net N$8: track 0.00 -> 22.8 mm
- net VOL_POT_SIG: track 0.00 -> 20.2 mm
- net AGND: track 0.00 -> 19.5 mm, vias 0 -> 2
- net BQ_LOAD_OUT: track 0.00 -> 18.7 mm
- net SCL_5V: track 0.00 -> 14.7 mm
- net N$21: track 0.00 -> 12.7 mm
- net N$19: track 0.00 -> 10.8 mm
- net N$30: track 0.00 -> 10.4 mm
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Other:
- board size 100 x 80 mm -> 97.5 x 62 mm
- board text added: "3.3"
- board text added: "3.3V"
- board text added: "5V"
- board text added: "5V+"
- board text added: "<GND"
- board text added: "<HYD_COM1"
- board text added: "BONE+"
- board text added: "BONE-"
- board text added: "BQ24074 Charger Controller"
- board text added: "CE"
- board text added: "CHG"
- board text added: "DOUT"
- board text added: "GND"
- board text added: "GNDBridge"
- board text added: "Green Team"
- board text added: "HYD+"
- board text added: "HYD-"
- board text added: "HYD_COM2>"
- board text added: "I2CV"
- board text added: "ISET"
- board text added: "It says: "you forgot to write in your lab notebook AGAIN" https://xkcd.com/1457/"
- board text added: "L+"
- board text added: "L-"
- board text added: "LBrg"
- board text added: "MCPWR"
- board text added: "MIT 2.009"
- board text added: "OUT"
- board text added: "OnOffButton"
- board text added: "PB_EN"
- board text added: "PGOOD"
- board text added: "PowerBoost 1000 Boost Converter"
- board text added: "R+"
- board text added: "R-"
- board text added: "RBrg"
- board text added: "RXGain Adj"
- board text added: "SCL"
- board text added: "SCL3V"
- board text added: "SCL5"
- board text added: "SCL5V"
- board text added: "SCLSEL 1(A) 0"
- board text added: "SDA"
- board text added: "SDA3V"
- board text added: "SDA5"
- board text added: "SDA5V"
- board text added: "SDASEL 1(A) 0"
- board text added: "SHDN"
- board text added: "THM"
- board text added: "TPA2016 Audio Amplifier"
- board text added: "TXRX>"
- board text added: "TXRX> SIG"
- board text added: "VB"
- board text added: "VBAT"
- board text added: "VBAT+"
- board text added: "VBUS"
- board text added: "VOL+"
- board text added: "VOLP"
- board text added: "VolumePot"
- board text added: "WCHG"
- board text added: "We got an underwater message!! But... it doesn't seem quite right..."
- board text added: "What came through??"

Commit message: done upper arm!!
Parts:
- removed JP9: JUMPER-SMT_2_NC_TRACE_NO-SILK, SparkFun-Jumpers:SMT-JUMPER_2_NC_TRACE_NO-SILK
- removed VR2: PT01-D115D-B103, SamacSys_Parts:PT01D115DB103
- added C11: 0.1uF, rcl:C0805
- added C12, C13, C14, C15, C18, C19, C20, C22, C23, C24, C25, C26, C28: 1uF, rcl:C0805
- added C27, C29: 10uF, rcl:C0805
- added VR1: 3310P-125-103L, SamacSys_Parts:3310P125103L
- moved SDAG 9.16 mm to (72.4, 66.2)
- moved C17 2.27 mm to (19.1, 42.0)
- moved HYD_TX_SIG 1.83 mm to (57.7, 30.3)
- moved D13 1.70 mm to (5.08, 34.2)
- moved IC4 1.20 mm to (52.5, 40.9)
- moved C2 0.65 mm to (49.2, 31.8)
- moved R4 0.40 mm to (51.5, 28.8)
- moved R12 0.28 mm to (44.0, 64.7)
- moved C9 0.15 mm to (25.5, 67.7), turned to 0 degrees
- moved S1 0.13 mm to (56.7, 45.7)
- moved R11 0.10 mm to (29.3, 67.8), turned to 180 degrees
- turned R13 to 180 degrees
Connections:
- removed net HYD_RX_IN2: K2.2
- removed net N$11: IC3.13, JP9.2
- net 3.3V: now also C28.2, C29.2, VR1.1; no longer VR2.1
- net 5V: now also C12.2, C13.2, C14.2, C15.2, C18.2, C19.2, C20.2, C22.2, C23.2, C24.2, C25.2, C26.2, C27.2
- net AGND: now also K2.2
- net GND: now also C11.2, C12.1, C13.1, C14.1, C15.1, C18.1, C19.1, C20.1, C22.1, C23.1, C24.1, C25.1, C26.1, C27.1, C28.1, C29.1, IC3.13, VR1.3; no longer JP9.1, VR2.3
- net N$5: now also IC2.3; no longer IC2.2
- net TXRX_RELAY: now also U$1.4
- net VBAT: now also C11.1, IC2.2; no longer IC2.3
- net VOL_POT_SIG: now also VR1.2; no longer VR2.2
Routing:
- net GND: track 173.4 -> 741.4 mm, vias 0 -> 5
- net 5V: track 138.4 -> 609.3 mm, vias 0 -> 12
- net 3.3V: track 25.3 -> 200.3 mm, vias 0 -> 8
- net BONECOND_-: track 0.00 -> 132.8 mm, vias 0 -> 6
- net BONECOND_+: track 0.00 -> 132.2 mm, vias 0 -> 5
- net TPA_R+: track 0.00 -> 98.2 mm, vias 0 -> 3
- net TPA_L+: track 0.00 -> 93.8 mm, vias 0 -> 3
- net TXRX_RELAY: track 0.00 -> 79.1 mm
- net HYD_TX_SIG: track 2.53 -> 72.2 mm, vias 0 -> 1
- net 3.3VI2C_SCL0: track 0.00 -> 63.3 mm, vias 0 -> 2
- net SCL_3V: track 6.51 -> 67.3 mm, vias 0 -> 2
- net 3.3VI2C_SDA0: track 0.00 -> 58.0 mm, vias 0 -> 2
- net 3.3VI2C_SCL1: track 0.00 -> 57.7 mm, vias 0 -> 4
- net SDA_3V: track 2.27 -> 59.4 mm, vias 0 -> 4
- net VBAT: track 33.4 -> 89.4 mm
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- added copper zone on layer 1, net AGND
- added copper zone on layer 1, net GND
- added copper zone on layer 16, net GND
Other:
- outline, holes or cut-outs redrawn
- board text added: "Designed by Aaron Becker, Nov 2024"
- board text added: "EN"
- board text added: "HSIG"
- board text added: "IN+"
- board text added: "LB"
- board text added: "powered by magik and caffeine"
- board text removed: "I2CV"
- board text removed: "MIT 2.009"
