File: UpperArmBoard/upperArm.sch (EAGLE design)
At the start: 2 parts

Commit message: nearly done!
Parts:
- added 3V, 5V, 5VG, BQ_USB_VBUS, HYD_COM1, HYD_COM2, HYD_RX_AMP, HYD_TX_SIG, SCLG, SCL_3V, SCL_5V, SDAG, SDA_3V, SDA_5V, TPA_L+, TPA_L-, TPA_R+, TPA_R-, TP_TXRX, VBAT, VBAT1: TPB1,27, testpad:TPB1,27
- added C1, C4, C6: 1uF, rcl:C-USC0805
- added C10: 10uF, microbuilder:CAP_CERAMIC0805
- added C16, C17: 9pF, rcl:C-USC0805
- added C2, C3: 10uF, rcl:C-USC0805
- added C21, C5: 0.1uF, rcl:C-USC0805
- added C7: 0.1µF, microbuilder:CAP_CERAMIC0805
- added C8: 0.01uF, microbuilder:CAP_CERAMIC0805
- added C9: 100pF, microbuilder:CAP_CERAMIC0805
- added D1, D10, D11, D13, D2, D3, D4, D5, D6, D7, D8, D9: WS2812_5050, SparkFun-LED:WS2812_5050
- added D12: SK34AQ-LTP, SamacSys_Parts:SK34AQ-LTP
- added FB2, FB3: BLM18PG471SN1D, SamacSys_Parts:BLM18PG471SN1D
- added IC1: LTC4311CSC6#TRPBF, SamacSys_Parts:LTC4311CSC6#TRPBF
- added IC2: MAX17048G+T10, SamacSys_Parts:MAX17048G+T10
- added IC3: PAM8904EGPR, SamacSys_Parts:PAM8904EGPR
- added IC4: DS04-254-2-02BK-SMT, SamacSys_Parts:DS04-254-2-02BK-SMT
- added J2, J3, J4: 1727052, SamacSys_Parts:1727052
- added JP11, JP12, JP13, JP7: (no value), pinhead:PINHD-1X1
- added JP14, JP2, JP3, JP8: JUMPER-SMT_3_1-NC_TRACE_NO-SILK, SparkFun-Jumpers:JUMPER-SMT_3_1-NC_TRACE_NO-SILK
- added JP4: (no value), pinhead:PINHD-1X6
- added JP5, JP6, JP9: JUMPER-SMT_2_NC_TRACE_NO-SILK, SparkFun-Jumpers:JUMPER-SMT_2_NC_TRACE_NO-SILK
- added K1, K2: G6K-2P-Y-DC5, SamacSys_Parts:G6K-2P-Y-DC5
- added LED2: RED, led:LEDCHIP-LED0805
- added Q1, Q2: CSD17575Q3, SamacSys_Parts:CSD17575Q3
- added Q3, Q4: BSS138, microbuilder:MOSFET-NWIDE
- added R1, R17, R18, R2, R3, R32, R4, R5: 10k, rcl:R-US_R0805
- added R10, R9: 1M, microbuilder:RESISTOR0805
- added R11: 22K, microbuilder:RESISTOR0805
- added R12: 3386P-1-104LF, 3386P-1-104LF:3386P-1-104LF
- added R13: 100, rcl:R-US_R0603
- added R14, R23: 220, rcl:R-US_R0805
- added R27: 100k, rcl:R-US_R0805
- added R29: 100, rcl:R-US_R0805
- added R6, R7, R8: 1K, microbuilder:RESISTOR0805
- added S1: GPTS203211B, SamacSys_Parts:GPTS203211B
- added U$11, U$14, U$15, U$16, U$17, U$18, U$19: MOUNTINGHOLE2.5, microbuilder:MOUNTINGHOLE2.5
- added U$7: (no value), pinhead:PINHD-1X10
- added U1: MAX4466EXK+T, microbuilder:MAX4466""
- added U8: BNO055, BNO055:BNO055
- added VR2: PT01-D115D-B103, SamacSys_Parts:PT01-D115D-B103
- added Y1: NDK_NX3215SA-32.768K-STD-MUA-9, NDK - NX3215SA-32.768K-STD-MUA-8:NDK_NX3215SA-32.768K-STD-MUA-8NDK_NX3215SA-32.768K-STD-MUA-8_0_0
Connections:
- removed net BQ_LIPO_IN: JP1.10
- new net 3.3V: 3V.TP, C5.1, J2.2, JP14.3, JP8.1, Q3.G, Q4.G, R2.2, R3.2, R32.2, U$1.3V, U$7.10, U8.VDD, U8.VDDIO, VR2.CCW
- new net 5V: 5V.TP, C3.1, D1.VCC, D10.VCC, D11.VCC, D13.VCC, D2.VCC, D3.VCC, D4.VCC, D5.VCC, D6.VCC, D7.VCC, D8.VCC, D9.VCC, IC1.VCC, IC3.VIN, IC4.NO_1, IC4.NO_2, J3.2, JP14.1, JP4.1, K1.+, K2.+, R1.2, R17.2, R18.2, U$1.5V, U$7.1
- new net AGND: C10.P$2, C7.P$2, FB2.1, R9.1, U1.GND
- new net AVCC: FB3.1, R10.2, R7.2, U1.VCC
- new net BONECOND_+: J2.5, JP7.1, TPA_L+.TP
- new net BONECOND_-: J2.6, JP11.1, TPA_L-.TP
- new net HYD_COM1: HYD_COM1.TP, J2.3, K1.COM_1
- new net HYD_COM2: HYD_COM2.TP, J2.4, K2.COM_1
- new net HYD_RX_IN1: C8.P$1, K1.NC_1, R6.1
- new net HYD_RX_IN2: K2.NC_1
- new net HYD_RX_INPUT: C9.P$1, HYD_RX_AMP.TP, R12.1, R12.2, U$1.MIC, U1.OUT
- new net HYD_TX_OUT1: IC3.VO2, K1.NO_1
- new net HYD_TX_OUT2: IC3.VO1, K2.NO_1
- new net HYD_TX_SIG: HYD_TX_SIG.TP, IC3.DIN, U$1.3
- new net IMU_CLK1: C16.2, U8.XIN32, Y1.1
- new net IMU_CLK2: C17.2, U8.XOUT32, Y1.2
- new net LED_BRIDGE: D6.DI, D8.DO
- new net LED_DIN: R13.1, U$1.2
- new net LED_DOUT: D11.DO, J3.5
- new net N$1: IC1.ENABLE, R1.1
- new net N$11: IC3.EP, JP9.2
- new net N$12: IC3.EN1, IC4.COM_2, R4.2
- new net N$13: IC3.EN2, IC4.COM_1, R5.1
- new net N$15: FB3.2, JP14.2
- new net N$16: C7.P$1, R6.2, R7.1
- new net N$17: C8.P$2, R10.1, R9.2, U1.IN+
- new net N$18: D1.DI, D13.DO
- new net N$19: C9.P$2, R11.1, R8.2, U1.IN-
- new net N$20: C10.P$1, R8.1
- new net N$21: R11.2, R12.3
- new net N$24: D12.A, J4.3
- new net N$25: D2.DO, D3.DI
- new net N$26: D3.DO, D4.DI
- new net N$27: D4.DO, D5.DI
- new net N$28: D5.DO, D8.DI
- new net N$29: D7.DO, D9.DI
- new net N$30: D10.DI, D9.DO
- new net N$31: D10.DO, D11.DI
- new net N$32: JP6.2, U$7.7
- new net N$37: C21.2, U8.CAP
- new net N$4: D6.DO, D7.DI
- new net N$40: R32.1, U8.NBOOT_LOAD_PIN
- new net N$5: IC2.CELL, JP8.2
- new net N$6: Q2.G, R14.2
- new net N$7: C2.1, IC3.VOUT
- new net N$81: Q1.G, R23.2
- new net N$82: LED2.A, R29.1
- new net NC_BCLK: U$1.21
- new net NC_DIN: U$1.7
- new net NC_DOUT: U$1.8
- new net NC_LRCLK: U$1.20
- new net NC_MCLK: U$1.23
- new net NC_MEMCS: U$1.6
- new net NC_MISO: U$1.12
- new net NC_MOSI: U$1.11
- new net NC_SCK: U$1.13
- new net NC_SDCS: U$1.10
- new net NC_VOL: U$1.15
- new net PAM_CN1: C4.2, IC3.CN1
- new net PAM_CN2: C6.2, IC3.CN2
- new net PAM_CP1: C4.1, IC3.CP1
- new net PAM_CP2: C6.1, IC3.CP2
- new net PB1K_EN: J4.5, JP4.4, S1.2
- new net PB1K_LB: JP4.3
- new net SCL_3V: IC2.SCL, JP3.2, Q4.S, R3.1, SCL_3V.TP, U$7.8, U8.COM1
- new net SCL_5V: IC1.BUS1, J3.4, Q4.D, R18.1, SCL_5V.TP
- new net SDA_3V: IC2.SDA, JP2.2, Q3.S, R2.1, SDA_3V.TP, U$7.9, U8.COM0
- new net SDA_5V: IC1.BUS2, J3.3, Q3.D, R17.1, SDA_5V.TP
- new net TPA_L+: U$1.OUTL, U$7.6
- new net TPA_R+: U$1.OUTR, U$7.5
- new net TPA_SHDN: U$7.3
- new net TXRX_OUT1: K1.-, Q1.D_1, Q1.D_2, Q1.D_3, Q1.D_4
- new net TXRX_OUT2: K2.-, Q2.D_1, Q2.D_2, Q2.D_3, Q2.D_4
- new net TXRX_RELAY: R14.1, R23.1, R27.1, R29.2, TP_TXRX.TP
- new net VBAT: C1.1, IC2.VDD, J4.1, JP1.10, JP8.3, VBAT.TP
- new net VOL_POT_SIG: J2.1, U$1.14, VR2.WIPER
- net 3.3VI2C_SCL0: now also JP3.3
- net 3.3VI2C_SCL1: now also JP3.1
- net 3.3VI2C_SDA0: now also JP2.3
- net 3.3VI2C_SDA1: now also JP2.1
- net BQ_LOAD_OUT: now also JP4.6
- net BQ_USB_VBUS: now also BQ_USB_VBUS.TP, D12.K
- net GND: now also 5VG.TP, C1.2, C16.1, C17.1, C2.2, C21.1, C3.2, C5.2, D1.GND, D10.GND, D11.GND, D13.GND, D2.GND, D3.GND, D4.GND, D5.GND, D6.GND, D7.GND, D8.GND, D9.GND, FB2.2, IC1.GND_1, IC1.GND_2, IC2.CTG, IC2.EP, IC2.GND, IC2.QSTRT, IC3.GND, J3.1, J3.6, J4.2, J4.4, J4.6, JP4.2, JP4.5, JP5.1, JP6.1, JP9.1, LED2.C, Q1.S_1, Q1.S_2, Q1.S_3, Q2.S_1, Q2.S_2, Q2.S_3, R27.2, R4.1, R5.2, S1.1, SCLG.TP, SDAG.TP, U$1.G, U$1.INGND1, U$1.INGND2, U$1.MIC_GND, U$1.OUTGND, U$7.2, U8.COM2, U8.COM3, U8.GND, U8.GNDIO, U8.PIN10, U8.PIN15, U8.PIN16, U8.PS0, U8.PS1, VBAT1.TP, VR2.CW
- net N$10: now also D1.DO, D2.DI; no longer U$1.VOL_3.3V
- net N$2: now also JP12.1, TPA_R+.TP; no longer U$1.5V
- net N$3: now also JP13.1, TPA_R-.TP; no longer U$1.G
- net N$8: now also D13.DI, R13.2; no longer U$1.VOL_GND
- net N$9: now also JP5.2, U$7.4; no longer U$1.VOL
Other:
- note added: "+1"
- note added: "= ~25-125x gain"
- note added: "Abs Orientation (Gyro, Accel, Mag) and Temp"
- note added: "Ferrite bead filtering"
- note added: "Gain ="
- note added: "I2C Level Shifting"
- note added: "I2C Selector Logic (normal/alternate pins)"
- note added: "Ind LED"
- note added: "LTC4311 Active Terminator"
- note added: "LiPo Input"
- note added: "Low pass F3db = 1/R5*C4*2pi"
- note added: "On/Off Button"
- note added: "Questions for DR: - what to do with low battery outputs (from BQ, MAX, boost)? - transistor on input of PAM? 0.5x VIN from datasheet - extended length header pins through teensy audio shield - noise immunity by doubling up relays? should double up relays - soldered pads or screw terminals? - pinout of cable I2C devices: - MAX1704 Pinouts: Bat+, Bat-, Pswitch1, Pswitch2, WirelessChg+, WirelessChg-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"
- note added: "R5"
- note added: "TXRX Relay"
- note added: "TXRX Relay 2"
- note added: "VR1+R7"
- note added: "Wireless Charger"
- note added: "nFet Relay Drive"
- note added: "→"
- moved on the sheet: JP1

Commit message: done upper arm!!
Parts:
- removed JP9: JUMPER-SMT_2_NC_TRACE_NO-SILK, SparkFun-Jumpers:JUMPER-SMT_2_NC_TRACE_NO-SILK
- removed VR2: PT01-D115D-B103, SamacSys_Parts:PT01-D115D-B103
- added C11: 0.1uF, rcl:C-USC0805
- added C12, C13, C14, C15, C18, C19, C20, C22, C23, C24, C25, C26, C28: 1uF, rcl:C-USC0805
- added C27, C29: 10uF, rcl:C-USC0805
- added VR1: 3310P-125-103L, SamacSys_Parts:3310P-125-103L
Connections:
- removed net HYD_RX_IN2: K2.NC_1
- removed net N$11: IC3.EP, JP9.2
- net 3.3V: now also C28.2, C29.2, VR1.CCW; no longer VR2.CCW
- net 5V: now also C12.2, C13.2, C14.2, C15.2, C18.2, C19.2, C20.2, C22.2, C23.2, C24.2, C25.2, C26.2, C27.2
- net AGND: now also K2.NC_1
- net GND: now also C11.2, C12.1, C13.1, C14.1, C15.1, C18.1, C19.1, C20.1, C22.1, C23.1, C24.1, C25.1, C26.1, C27.1, C28.1, C29.1, IC3.EP, VR1.CW; no longer JP9.1, VR2.CW
- net N$5: now also IC2.VDD; no longer IC2.CELL
- net TXRX_RELAY: now also U$1.4
- net VBAT: now also C11.1, IC2.CELL; no longer IC2.VDD
- net VOL_POT_SIG: now also VR1.WIPER; no longer VR2.WIPER
Other:
- moved on the sheet: C2, JP8, VBAT
